File: untitled.kicad_sch (KiCad schematic)
At the start: 15 parts, among them U2 AMS1117-3.3, U4 TPS54336ADDA

Commit message: started layout
in meeting
Parts:
- removed BT1, BT2: 9V, symbol Device:Battery
- removed C1, C5: 10nF, symbol Device:C_Small
- removed C6: .1µF, symbol Device:C_Small
- removed C7: 5.6nF, symbol Device:C_Small
- removed C8: 100nF, symbol Device:C_Small
- removed C9: 44µF, symbol Device:C_Small
- removed F1: 2A 12V PTC fuse, symbol Device:Fuse
- removed L1: 4.7µH, symbol Device:L_Small
- removed R3: 25kΩ, symbol Device:R_Small_US
- removed R4: 10kΩ, symbol Device:R_Small_US
- removed R5: 100kΩ, symbol Device:R_Small_US
- removed U2: AMS1117-3.3, Package_TO_SOT_SMD:SOT-223-3_TabPin2, symbol Regulator_Linear:AMS1117-3.3
- removed U4: TPS54336ADDA, Package_SO:TI_SO-PowerPAD-8_ThermalVias, symbol Regulator_Switching:TPS54336ADDA
