File: USB-C.kicad_sch (KiCad schematic)
At the start: 5 parts, among them J1 USB4220-03-1040-C_REVA

Commit message: todolist update
update of the to do list on schematic
Changed lines of the file:
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@@
 	)
 	(hierarchical_label "USB-C_VBUS_A"
-		(shape input)
+		(shape output)
 		(at 95.25 25.4 0)
 		(effects
@@
 	)
 	(hierarchical_label "USB-C_DN2"
-		(shape input)
+		(shape output)
 		(at 95.25 45.72 0)
 		(effects
@@
 	)
 	(hierarchical_label "USB-C_DP2"
-		(shape input)
+		(shape output)
 		(at 95.25 48.26 0)
 		(effects

Commit message: USB, TVS, LDO, Passives, I2C
applied changes to usb circuitry, tvs, ldo, passibes and i2c.
Parts:
- removed J1: USB4220-03-1040-C_REVA, usbc:GCT_USB4220-03-1040-C_REVA, symbol usbc:USB4220-03-1040-C_REVA
- removed R_PD_USBC_1: 5.1k, Resistor_SMD:R_0603_1608Metric, symbol Device:R_Small_US
- removed R_PD_USBC_2: 5.1kΩ, Resistor_SMD:R_0603_1608Metric, symbol Device:R_Small_US
- removed R_USBC_DIV1: 20kΩ, Resistor_SMD:R_0603_1608Metric, symbol Device:R_Small_US
- removed R_USBC_DIV2: 10kΩ, Resistor_SMD:R_0603_1608Metric, symbol Device:R_Small_US
